File: signal_generator/signal_generator.sch (KiCad schematic (older format))
At the start: 32 parts, among them J101 DAC_OUT_BUF, J102 DAC_OUT, U101 Digilent_CMOD-S7_25, U102 ADC9765, U103 TL074

Commit message: send to production
Connections:
- net GNDA: now also R113.2, R114.2
- net at R113.1, U103.9 (-): now also R117.2
- net at R114.1, U103.13 (-): now also R118.2
Other:
- moved on the sheet: J101, R113, R114, R117, R118, RV103, RV104, U103C, U103D
Changed lines of the file:
@@
 L signal_generator-rescue:TL074-Amplifier_Operational U103
 U 3 1 5F9E0201
-P 9150 5050
-F 0 "U103" H 9150 5417 50  0000 C CNN
-F 1 "TL074" H 9150 5326 50  0000 C CNN
-F 2 "Package_SO:SOIC-14_3.9x8.7mm_P1.27mm" H 9100 5150 50  0001 C CNN
-F 3 "http://www.ti.com/lit/ds/symlink/tl071.pdf" H 9200 5250 50  0001 C CNN
-	3    9150 5050
+P 9350 4850
+F 0 "U103" H 9350 5217 50  0000 C CNN
+F 1 "TL074" H 9350 5126 50  0000 C CNN
+F 2 "Package_SO:SOIC-14_3.9x8.7mm_P1.27mm" H 9300 4950 50  0001 C CNN
+F 3 "http://www.ti.com/lit/ds/symlink/tl071.pdf" H 9400 5050 50  0001 C CNN
+	3    9350 4850
 	1    0    0    -1
 $EndComp
@@
 L signal_generator-rescue:TL074-Amplifier_Operational U103
 U 4 1 5F9E33AC
-P 9150 6000
-F 0 "U103" H 9150 6367 50  0000 C CNN
-F 1 "TL074" H 9150 6276 50  0000 C CNN
-F 2 "Package_SO:SOIC-14_3.9x8.7mm_P1.27mm" H 9100 6100 50  0001 C CNN
-F 3 "http://www.ti.com/lit/ds/symlink/tl071.pdf" H 9200 6200 50  0001 C CNN
-	4    9150 6000
+P 9350 5800
+F 0 "U103" H 9350 6167 50  0000 C CNN
+F 1 "TL074" H 9350 6076 50  0000 C CNN
+F 2 "Package_SO:SOIC-14_3.9x8.7mm_P1.27mm" H 9300 5900 50  0001 C CNN
+F 3 "http://www.ti.com/lit/ds/symlink/tl071.pdf" H 9400 6000 50  0001 C CNN
+	4    9350 5800
 	1    0    0    -1
 $EndComp
@@
 Wire Wire Line
 	5850 2650 5850 2700
-Text Label 8200 4700 2    50   ~ 0
+Text Label 8400 4500 2    50   ~ 0
 DAC_OUT1
 Wire Wire Line
@@
 L signal_generator-rescue:R_POT-Device RV103
 U 1 1 5FA7BAE5
-P 8450 4950
-F 0 "RV103" H 8380 4996 50  0000 R CNN
-F 1 "10kA" H 8380 4905 50  0000 R CNN
-F 2 "Potentiometer_THT:Potentiometer_Alpha_RD901F-40-00D_Single_Vertical_CircularHoles" H 8450 4950 50  0001 C CNN
-F 3 "~" H 8450 4950 50  0001 C CNN
-	1    8450 4950
+P 8650 4750
+F 0 "RV103" H 8580 4796 50  0000 R CNN
+F 1 "10kA" H 8580 4705 50  0000 R CNN
+F 2 "Potentiometer_THT:Potentiometer_Alpha_RD901F-40-00D_Single_Vertical_CircularHoles" H 8650 4750 50  0001 C CNN
+F 3 "~" H 8650 4750 50  0001 C CNN
+	1    8650 4750
 	1    0    0    -1
 $EndComp
@@
 $EndComp
 Wire Wire Line
-	8600 4950 8850 4950
-Wire Wire Line
-	8450 4800 8450 4700
-Wire Wire Line
-	8450 4700 8200 4700
+	8800 4750 9050 4750
+Wire Wire Line
+	8650 4600 8650 4500
+Wire Wire Line
+	8650 4500 8400 4500
 $Comp
 L signal_generator-rescue:GNDA-power #PWR0116
 U 1 1 5FBC8950
-P 8450 5200
-F 0 "#PWR0116" H 8450 4950 50  0001 C CNN
-F 1 "GNDA" H 8455 5027 50  0000 C CNN
-F 2 "" H 8450 5200 50  0001 C CNN
-F 3 "" H 8450 5200 50  0001 C CNN
-	1    8450 5200
-	1    0    0    -1
-$EndComp
-Wire Wire Line
-	8450 5200 8450 5100
+P 8650 5000
+F 0 "#PWR0116" H 8650 4750 50  0001 C CNN
+F 1 "GNDA" H 8655 4827 50  0000 C CNN
+F 2 "" H 8650 5000 50  0001 C CNN
+F 3 "" H 8650 5000 50  0001 C CNN
+	1    8650 5000
+	1    0    0    -1
+$EndComp
+Wire Wire Line
+	8650 5000 8650 4900
 $Comp
 L signal_generator-rescue:R_Small-Device R113
 U 1 1 5FBD6E96
-P 8750 5300
-F 0 "R113" H 8809 5346 50  0000 L CNN
-F 1 "R_Small" H 8809 5255 50  0000 L CNN
-F 2 "Resistor_SMD:R_0603_1608Metric_Pad0.98x0.95mm_HandSolder" H 8750 5300 50  0001 C CNN
-F 3 "~" H 8750 5300 50  0001 C CNN
-	1    8750 5300
+P 8950 5350
+F 0 "R113" H 9009 5396 50  0000 L CNN
+F 1 "R_Small" H 9009 5305 50  0000 L CNN
+F 2 "Resistor_SMD:R_0603_1608Metric_Pad0.98x0.95mm_HandSolder" H 8950 5350 50  0001 C CNN
+F 3 "~" H 8950 5350 50  0001 C CNN
+	1    8950 5350
 	1    0    0    -1
 $EndComp
@@
 L signal_generator-rescue:R_Small-Device R117
 U 1 1 5FBD7707
-P 9350 5450
-F 0 "R117" V 9154 5450 50  0000 C CNN
-F 1 "R_Small" V 9245 5450 50  0000 C CNN
-F 2 "Resistor_SMD:R_0603_1608Metric_Pad0.98x0.95mm_HandSolder" H 9350 5450 50  0001 C CNN
-F 3 "~" H 9350 5450 50  0001 C CNN
-	1    9350 5450
+P 9550 5250
+F 0 "R117" V 9354 5250 50  0000 C CNN
+F 1 "R_Small" V 9445 5250 50  0000 C CNN
+F 2 "Resistor_SMD:R_0603_1608Metric_Pad0.98x0.95mm_HandSolder" H 9550 5250 50  0001 C CNN
+F 3 "~" H 9550 5250 50  0001 C CNN
+	1    9550 5250
 	0    1    1    0
 $EndComp
 Wire Wire Line
-	9250 5450 8750 5450
-Wire Wire Line
-	8750 5450 8750 5400
-Wire Wire Line
-	8750 5200 8750 5150
-Wire Wire Line
-	8750 5150 8850 5150
-Wire Wire Line
-	9450 5450 9550 5450
-Wire Wire Line
-	9550 5450 9550 5050
-Wire Wire Line
-	9550 5050 9450 5050
-Connection ~ 9550 5050
+	8950 4950 9050 4950
+Wire Wire Line
+	9650 5250 9750 5250
+Wire Wire Line
+	9750 5250 9750 4850
+Wire Wire Line
+	9750 4850 9650 4850
+Connection ~ 9750 4850
 $Comp
 L signal_generator-rescue:R_POT-Device RV104
 U 1 1 5FC29F19
-P 8450 5900
-F 0 "RV104" H 8380 5946 50  0000 R CNN
-F 1 "10kA" H 8380 5855 50  0000 R CNN
-F 2 "Potentiometer_THT:Potentiometer_Alpha_RD901F-40-00D_Single_Vertical_CircularHoles" H 8450 5900 50  0001 C CNN
-F 3 "~" H 8450 5900 50  0001 C CNN
-	1    8450 5900
-	1    0    0    -1
-$EndComp
-Wire Wire Line
-	8600 5900 8850 5900
-Wire Wire Line
-	8450 5750 8450 5650
-Wire Wire Line
-	8450 5650 8200 5650
+P 8650 5700
+F 0 "RV104" H 8580 5746 50  0000 R CNN
+F 1 "10kA" H 8580 5655 50  0000 R CNN
+F 2 "Potentiometer_THT:Potentiometer_Alpha_RD901F-40-00D_Single_Vertical_CircularHoles" H 8650 5700 50  0001 C CNN
+F 3 "~" H 8650 5700 50  0001 C CNN
+	1    8650 5700
+	1    0    0    -1
+$EndComp
+Wire Wire Line
+	8800 5700 9050 5700
+Wire Wire Line
+	8650 5550 8650 5450
+Wire Wire Line
+	8650 5450 8400 5450
 $Comp
 L signal_generator-rescue:GNDA-power #PWR0117
 U 1 1 5FC29F22
-P 8450 6150
-F 0 "#PWR0117" H 8450 5900 50  0001 C CNN
-F 1 "GNDA" H 8455 5977 50  0000 C CNN
-F 2 "" H 8450 6150 50  0001 C CNN
-F 3 "" H 8450 6150 50  0001 C CNN
-	1    8450 6150
-	1    0    0    -1
-$EndComp
-Wire Wire Line
-	8450 6150 8450 6050
+P 8650 5950
+F 0 "#PWR0117" H 8650 5700 50  0001 C CNN
+F 1 "GNDA" H 8655 5777 50  0000 C CNN
+F 2 "" H 8650 5950 50  0001 C CNN
+F 3 "" H 8650 5950 50  0001 C CNN
+	1    8650 5950
+	1    0    0    -1
+$EndComp
+Wire Wire Line
+	8650 5950 8650 5850
 $Comp
 L signal_generator-rescue:R_Small-Device R114
 U 1 1 5FC29F29
-P 8750 6250
-F 0 "R114" H 8809 6296 50  0000 L CNN
-F 1 "R_Small" H 8809 6205 50  0000 L CNN
-F 2 "Resistor_SMD:R_0603_1608Metric_Pad0.98x0.95mm_HandSolder" H 8750 6250 50  0001 C CNN
-F 3 "~" H 8750 6250 50  0001 C CNN
-	1    8750 6250
+P 8950 6300
+F 0 "R114" H 9009 6346 50  0000 L CNN
+F 1 "R_Small" H 9009 6255 50  0000 L CNN
+F 2 "Resistor_SMD:R_0603_1608Metric_Pad0.98x0.95mm_HandSolder" H 8950 6300 50  0001 C CNN
+F 3 "~" H 8950 6300 50  0001 C CNN
+	1    8950 6300
 	1    0    0    -1
 $EndComp
@@
 L signal_generator-rescue:R_Small-Device R118
 U 1 1 5FC29F2F
-P 9350 6400
-F 0 "R118" V 9154 6400 50  0000 C CNN
-F 1 "R_Small" V 9245 6400 50  0000 C CNN
-F 2 "Resistor_SMD:R_0603_1608Metric_Pad0.98x0.95mm_HandSolder" H 9350 6400 50  0001 C CNN
-F 3 "~" H 9350 6400 50  0001 C CNN
-	1    9350 6400
+P 9550 6200
+F 0 "R118" V 9354 6200 50  0000 C CNN
+F 1 "R_Small" V 9445 6200 50  0000 C CNN
+F 2 "Resistor_SMD:R_0603_1608Metric_Pad0.98x0.95mm_HandSolder" H 9550 6200 50  0001 C CNN
+F 3 "~" H 9550 6200 50  0001 C CNN
+	1    9550 6200
 	0    1    1    0
 $EndComp
 Wire Wire Line
-	9250 6400 8750 6400
-Wire Wire Line
-	8750 6400 8750 6350
-Wire Wire Line
-	8750 6150 8750 6100
-Wire Wire Line
-	8750 6100 8850 6100
-Wire Wire Line
-	9450 6400 9550 6400
-Wire Wire Line
-	9550 6400 9550 6000
-Wire Wire Line
-	9550 6000 9450 6000
-Connection ~ 9550 6000
-Text Label 8200 5650 2    50   ~ 0
+	8950 5900 9050 5900
+Wire Wire Line
+	9650 6200 9750 6200
+Wire Wire Line
+	9750 6200 9750 5800
+Wire Wire Line
+	9750 5800 9650 5800
+Connection ~ 9750 5800
+Text Label 8400 5450 2    50   ~ 0
 DAC_OUT2
-Text Label 9700 5050 1    50   ~ 0
+Text Label 9900 4850 1    50   ~ 0
 DAC_OUT1_BUF
-Text Label 9700 6000 1    50   ~ 0
+Text Label 9900 5800 1    50   ~ 0
 DAC_OUT2_BUF
 $Comp
 L signal_generator-rescue:Conn_01x02_Male-Connector J101
 U 1 1 5FD80DC5
-P 10300 5500
-F 0 "J101" H 10272 5474 50  0000 R CNN
-F 1 "DAC_OUT_BUF" H 10272 5383 50  0000 R CNN
-F 2 "Connector_PinHeader_2.54mm:PinHeader_1x02_P2.54mm_Vertical" H 10300 5500 50  0001 C CNN
-F 3 "~" H 10300 5500 50  0001 C CNN
-	1    10300 5500
+P 10500 5300
+F 0 "J101" H 10472 5274 50  0000 R CNN
+F 1 "DAC_OUT_BUF" H 10472 5183 50  0000 R CNN
+F 2 "Connector_PinHeader_2.54mm:PinHeader_1x02_P2.54mm_Vertical" H 10500 5300 50  0001 C CNN
+F 3 "~" H 10500 5300 50  0001 C CNN
+	1    10500 5300
 	-1   0    0    -1
 $EndComp
 Wire Wire Line
-	10000 5050 10000 5500
-Wire Wire Line
-	9550 5050 10000 5050
-Wire Wire Line
-	10000 5600 10000 6000
-Wire Wire Line
-	9550 6000 10000 6000
-Wire Wire Line
-	10000 5500 10100 5500
-Wire Wire Line
-	10000 5600 10100 5600
+	10200 4850 10200 5300
+Wire Wire Line
+	9750 4850 10200 4850
+Wire Wire Line
+	10200 5400 10200 5800
+Wire Wire Line
+	9750 5800 10200 5800
+Wire Wire Line
+	10200 5300 10300 5300
+Wire Wire Line
+	10200 5400 10300 5400
 $Sheet
 S 1100 950  1100 1750
@@
 Wire Wire Line
 	9950 2950 9950 3600
+Wire Wire Line
+	9450 6200 8950 6200
+Wire Wire Line
+	8950 5900 8950 6200
+Wire Wire Line
+	8950 5250 9450 5250
+Wire Wire Line
+	8950 4950 8950 5250
+$Comp
+L signal_generator-rescue:GNDA-power #PWR?
+U 1 1 5FACA75C
+P 8950 5500
+F 0 "#PWR?" H 8950 5250 50  0001 C CNN
+F 1 "GNDA" H 8955 5327 50  0000 C CNN
+F 2 "" H 8950 5500 50  0001 C CNN
+F 3 "" H 8950 5500 50  0001 C CNN
+	1    8950 5500
+	1    0    0    -1
+$EndComp
+Connection ~ 8950 6200
+$Comp
+L signal_generator-rescue:GNDA-power #PWR?
+U 1 1 5FB00D9A
+P 8950 6450
+F 0 "#PWR?" H 8950 6200 50  0001 C CNN
+F 1 "GNDA" H 8955 6277 50  0000 C CNN
+F 2 "" H 8950 6450 50  0001 C CNN
+F 3 "" H 8950 6450 50  0001 C CNN
+	1    8950 6450
+	1    0    0    -1
+$EndComp
+Wire Wire Line
+	8950 6450 8950 6400
+Connection ~ 8950 5250
+Wire Wire Line
+	8950 5500 8950 5450
 $EndSCHEMATC

Commit message: final status
Parts:
- R101, R102: value 256 -> 240R
- R105, R106, R107, R108: value 25R -> 27R
- R109, R110, R111, R112: value 225R -> 2k2
- R113, R114, R117, R118: value R_Small -> 10k
- R115, R116: value 500R -> 4k7
- U103: value TL074 -> TL074/TLV3544
Changed lines of the file:
@@
 P 8750 2100
 F 0 "R109" V 8554 2100 50  0000 C CNN
-F 1 "225R" V 8645 2100 50  0000 C CNN
+F 1 "2k2" V 8645 2100 50  0000 C CNN
 F 2 "Resistor_SMD:R_0603_1608Metric_Pad0.98x0.95mm_HandSolder" H 8750 2100 50  0001 C CNN
 F 3 "~" H 8750 2100 50  0001 C CNN
@@
 P 8750 2300
 F 0 "R110" V 8650 2300 50  0000 C CNN
-F 1 "225R" V 8850 2300 50  0000 C CNN
+F 1 "2k2" V 8850 2300 50  0000 C CNN
 F 2 "Resistor_SMD:R_0603_1608Metric_Pad0.98x0.95mm_HandSolder" H 8750 2300 50  0001 C CNN
 F 3 "~" H 8750 2300 50  0001 C CNN
@@
 P 8150 2550
 F 0 "R105" H 8209 2596 50  0000 L CNN
-F 1 "25R" H 8209 2505 50  0000 L CNN
+F 1 "27R" H 8209 2505 50  0000 L CNN
 F 2 "Resistor_SMD:R_0603_1608Metric_Pad0.98x0.95mm_HandSolder" H 8150 2550 50  0001 C CNN
 F 3 "~" H 8150 2550 50  0001 C CNN
@@
 P 8450 2550
 F 0 "R107" H 8509 2596 50  0000 L CNN
-F 1 "25R" H 8509 2505 50  0000 L CNN
+F 1 "27R" H 8509 2505 50  0000 L CNN
 F 2 "Resistor_SMD:R_0603_1608Metric_Pad0.98x0.95mm_HandSolder" H 8450 2550 50  0001 C CNN
 F 3 "~" H 8450 2550 50  0001 C CNN
@@
 Wire Wire Line
 	9050 2100 8950 2100
-Wire Wire Line
-	8850 2300 9050 2300
 Wire Wire Line
 	8650 2300 8150 2300
@@
 P 9350 1650
 F 0 "R115" V 9154 1650 50  0000 C CNN
-F 1 "500R" V 9245 1650 50  0000 C CNN
+F 1 "4k7" V 9245 1650 50  0000 C CNN
 F 2 "Resistor_SMD:R_0603_1608Metric_Pad0.98x0.95mm_HandSolder" H 9350 1650 50  0001 C CNN
 F 3 "~" H 9350 1650 50  0001 C CNN
@@
 P 8750 3500
 F 0 "R111" V 8554 3500 50  0000 C CNN
-F 1 "225R" V 8645 3500 50  0000 C CNN
+F 1 "2k2" V 8645 3500 50  0000 C CNN
 F 2 "Resistor_SMD:R_0603_1608Metric_Pad0.98x0.95mm_HandSolder" H 8750 3500 50  0001 C CNN
 F 3 "~" H 8750 3500 50  0001 C CNN
@@
 P 8750 3700
 F 0 "R112" V 8650 3700 50  0000 C CNN
-F 1 "225R" V 8850 3700 50  0000 C CNN
+F 1 "2k2" V 8850 3700 50  0000 C CNN
 F 2 "Resistor_SMD:R_0603_1608Metric_Pad0.98x0.95mm_HandSolder" H 8750 3700 50  0001 C CNN
 F 3 "~" H 8750 3700 50  0001 C CNN
@@
 P 8150 3950
 F 0 "R106" H 8209 3996 50  0000 L CNN
-F 1 "25R" H 8209 3905 50  0000 L CNN
+F 1 "27R" H 8209 3905 50  0000 L CNN
 F 2 "Resistor_SMD:R_0603_1608Metric_Pad0.98x0.95mm_HandSolder" H 8150 3950 50  0001 C CNN
 F 3 "~" H 8150 3950 50  0001 C CNN
@@
 P 8450 3950
 F 0 "R108" H 8509 3996 50  0000 L CNN
-F 1 "25R" H 8509 3905 50  0000 L CNN
+F 1 "27R" H 8509 3905 50  0000 L CNN
 F 2 "Resistor_SMD:R_0603_1608Metric_Pad0.98x0.95mm_HandSolder" H 8450 3950 50  0001 C CNN
 F 3 "~" H 8450 3950 50  0001 C CNN
@@
 Wire Wire Line
 	9050 3500 8950 3500
-Wire Wire Line
-	8850 3700 9050 3700
 Wire Wire Line
 	8650 3700 8150 3700
@@
 P 9350 3050
 F 0 "R116" V 9154 3050 50  0000 C CNN
-F 1 "500R" V 9245 3050 50  0000 C CNN
+F 1 "4k7" V 9245 3050 50  0000 C CNN
 F 2 "Resistor_SMD:R_0603_1608Metric_Pad0.98x0.95mm_HandSolder" H 9350 3050 50  0001 C CNN
 F 3 "~" H 9350 3050 50  0001 C CNN
@@
 P 4950 3000
 F 0 "R102" H 5020 3046 50  0000 L CNN
-F 1 "256" H 5020 2955 50  0000 L CNN
+F 1 "240R" H 5020 2955 50  0000 L CNN
 F 2 "Resistor_SMD:R_0603_1608Metric_Pad0.98x0.95mm_HandSolder" V 4880 3000 50  0001 C CNN
 F 3 "~" H 4950 3000 50  0001 C CNN
@@
 P 4550 4700
 F 0 "R101" H 4620 4746 50  0000 L CNN
-F 1 "256" H 4620 4655 50  0000 L CNN
+F 1 "240R" H 4620 4655 50  0000 L CNN
 F 2 "Resistor_SMD:R_0603_1608Metric_Pad0.98x0.95mm_HandSolder" V 4480 4700 50  0001 C CNN
 F 3 "~" H 4550 4700 50  0001 C CNN
@@
 P 9350 2200
 F 0 "U103" H 9350 1833 50  0000 C CNN
-F 1 "TL074" H 9350 1924 50  0000 C CNN
+F 1 "TL074/TLV3544" H 9350 1924 50  0000 C CNN
 F 2 "Package_SO:SOIC-14_3.9x8.7mm_P1.27mm" H 9300 2300 50  0001 C CNN
 F 3 "http://www.ti.com/lit/ds/symlink/tl071.pdf" H 9400 2400 50  0001 C CNN
@@
 P 9350 3600
 F 0 "U103" H 9350 3233 50  0000 C CNN
-F 1 "TL074" H 9350 3324 50  0000 C CNN
+F 1 "TL074/TLV3544" H 9350 3324 50  0000 C CNN
 F 2 "Package_SO:SOIC-14_3.9x8.7mm_P1.27mm" H 9300 3700 50  0001 C CNN
 F 3 "http://www.ti.com/lit/ds/symlink/tl071.pdf" H 9400 3800 50  0001 C CNN
@@
 P 9350 4850
 F 0 "U103" H 9350 5217 50  0000 C CNN
-F 1 "TL074" H 9350 5126 50  0000 C CNN
+F 1 "TL074/TLV3544" H 9350 5126 50  0000 C CNN
 F 2 "Package_SO:SOIC-14_3.9x8.7mm_P1.27mm" H 9300 4950 50  0001 C CNN
 F 3 "http://www.ti.com/lit/ds/symlink/tl071.pdf" H 9400 5050 50  0001 C CNN
@@
 P 9350 5800
 F 0 "U103" H 9350 6167 50  0000 C CNN
-F 1 "TL074" H 9350 6076 50  0000 C CNN
+F 1 "TL074/TLV3544" H 9350 6076 50  0000 C CNN
 F 2 "Package_SO:SOIC-14_3.9x8.7mm_P1.27mm" H 9300 5900 50  0001 C CNN
 F 3 "http://www.ti.com/lit/ds/symlink/tl071.pdf" H 9400 6000 50  0001 C CNN
@@
 P 8950 5350
 F 0 "R113" H 9009 5396 50  0000 L CNN
-F 1 "R_Small" H 9009 5305 50  0000 L CNN
+F 1 "10k" H 9009 5305 50  0000 L CNN
 F 2 "Resistor_SMD:R_0603_1608Metric_Pad0.98x0.95mm_HandSolder" H 8950 5350 50  0001 C CNN
 F 3 "~" H 8950 5350 50  0001 C CNN
@@
 P 9550 5250
 F 0 "R117" V 9354 5250 50  0000 C CNN
-F 1 "R_Small" V 9445 5250 50  0000 C CNN
+F 1 "10k" V 9445 5250 50  0000 C CNN
 F 2 "Resistor_SMD:R_0603_1608Metric_Pad0.98x0.95mm_HandSolder" H 9550 5250 50  0001 C CNN
 F 3 "~" H 9550 5250 50  0001 C CNN
@@
 P 8950 6300
 F 0 "R114" H 9009 6346 50  0000 L CNN
-F 1 "R_Small" H 9009 6255 50  0000 L CNN
+F 1 "10k" H 9009 6255 50  0000 L CNN
 F 2 "Resistor_SMD:R_0603_1608Metric_Pad0.98x0.95mm_HandSolder" H 8950 6300 50  0001 C CNN
 F 3 "~" H 8950 6300 50  0001 C CNN
@@
 P 9550 6200
 F 0 "R118" V 9354 6200 50  0000 C CNN
-F 1 "R_Small" V 9445 6200 50  0000 C CNN
+F 1 "10k" V 9445 6200 50  0000 C CNN
 F 2 "Resistor_SMD:R_0603_1608Metric_Pad0.98x0.95mm_HandSolder" H 9550 6200 50  0001 C CNN
 F 3 "~" H 9550 6200 50  0001 C CNN
@@
 	8950 4950 8950 5250
 $Comp
-L signal_generator-rescue:GNDA-power #PWR?
+L signal_generator-rescue:GNDA-power #PWR0122
 U 1 1 5FACA75C
 P 8950 5500
-F 0 "#PWR?" H 8950 5250 50  0001 C CNN
+F 0 "#PWR0122" H 8950 5250 50  0001 C CNN
 F 1 "GNDA" H 8955 5327 50  0000 C CNN
 F 2 "" H 8950 5500 50  0001 C CNN
@@
 Connection ~ 8950 6200
 $Comp
-L signal_generator-rescue:GNDA-power #PWR?
+L signal_generator-rescue:GNDA-power #PWR0123
 U 1 1 5FB00D9A
 P 8950 6450
-F 0 "#PWR?" H 8950 6200 50  0001 C CNN
+F 0 "#PWR0123" H 8950 6200 50  0001 C CNN
 F 1 "GNDA" H 8955 6277 50  0000 C CNN
 F 2 "" H 8950 6450 50  0001 C CNN
@@
 Wire Wire Line
 	8950 5500 8950 5450
+Wire Wire Line
+	8850 3700 9050 3700
+Wire Wire Line
+	8850 2300 9050 2300
 $EndSCHEMATC
