File: signal_generator/supply.sch (KiCad schematic (older format))
At the start: 30 parts, among them J201 Power Input, J202 Power Output, U103 TL074, U201 TPS76933, U202 LM2611, U203 TPS76901, U204 TPS72301

Commit message: finished PCB v1
Parts:
- C201, C206, C212, C213: symbol Device:CP_Small -> signal_generator-rescue:CP_Small-Device
- C202, C209, C210, C211: symbol Device:C_Small -> signal_generator-rescue:C_Small-Device
- C203, C204, C205, C207, C208: footprint Capacitor_SMD:C_0603_1608Metric -> Capacitor_SMD:C_0603_1608Metric_Pad1.08x0.95mm_HandSolder; symbol Device:C_Small -> signal_generator-rescue:C_Small-Device
- D201: symbol Diode:MBR0520LT -> signal_generator-rescue:MBR0520LT-Diode
- J201: symbol Connector:Conn_01x02_Male -> signal_generator-rescue:Conn_01x02_Male-Connector
- J202: symbol Connector:Conn_01x05_Male -> signal_generator-rescue:Conn_01x05_Male-Connector
- L201, L202: symbol Device:L_Small -> signal_generator-rescue:L_Small-Device
- L203: footprint Inductor_SMD:L_0805_2012Metric -> Inductor_THT:L_Axial_L7.0mm_D3.3mm_P10.16mm_Horizontal_Fastron_MICC; symbol Device:L_Small -> signal_generator-rescue:L_Small-Device
- R201, R202, R203, R204, R205, R206: symbol Device:R_Small -> signal_generator-rescue:R_Small-Device
- U103: footprint Package_SO:SSOP-14_5.3x6.2mm_P0.65mm -> Package_SO:SOIC-14_3.9x8.7mm_P1.27mm; symbol Amplifier_Operational:TL074 -> signal_generator-rescue:TL074-Amplifier_Operational
- U201: symbol Regulator_Linear:TPS76933 -> signal_generator-rescue:TPS76933-Regulator_Linear
- U203: symbol Regulator_Linear:TPS76901 -> signal_generator-rescue:TPS76901-Regulator_Linear
Connections:
- net -5VA is gone; now on net VSSA: C204.2, U103.11 (V-)

Commit message: final status
Parts:
- R203: value 30k -> 360k
- R204: value 30k -> 150k
- R205: value 30k -> 68k
- R206: value 30k -> 27k
- U103: value TL074 -> TL074/TLV3544
Changed lines of the file:
@@
 P 8150 2250
 F 0 "R205" H 8209 2296 50  0000 L CNN
-F 1 "30k" H 8209 2205 50  0000 L CNN
+F 1 "68k" H 8209 2205 50  0000 L CNN
 F 2 "DSC-Supply:C0805" H 8150 2250 50  0001 C CNN
 F 3 "~" H 8150 2250 50  0001 C CNN
@@
 P 8150 2600
 F 0 "R206" H 8209 2646 50  0000 L CNN
-F 1 "30k" H 8209 2555 50  0000 L CNN
+F 1 "27k" H 8209 2555 50  0000 L CNN
 F 2 "DSC-Supply:C0805" H 8150 2600 50  0001 C CNN
 F 3 "~" H 8150 2600 50  0001 C CNN
@@
 P 5550 2150
 F 0 "R203" H 5609 2196 50  0000 L CNN
-F 1 "30k" H 5609 2105 50  0000 L CNN
+F 1 "360k" H 5609 2105 50  0000 L CNN
 F 2 "DSC-Supply:C0805" H 5550 2150 50  0001 C CNN
 F 3 "~" H 5550 2150 50  0001 C CNN
@@
 P 5550 2500
 F 0 "R204" H 5609 2546 50  0000 L CNN
-F 1 "30k" H 5609 2455 50  0000 L CNN
+F 1 "150k" H 5609 2455 50  0000 L CNN
 F 2 "DSC-Supply:C0805" H 5550 2500 50  0001 C CNN
 F 3 "~" H 5550 2500 50  0001 C CNN
@@
 AR Path="/5FA42535/5FBC15F6" Ref="U103"  Part="5"
 F 0 "U103" H 1658 6696 50  0000 L CNN
-F 1 "TL074" H 1658 6605 50  0000 L CNN
+F 1 "TL074/TLV3544" H 1658 6605 50  0000 L CNN
 F 2 "Package_SO:SOIC-14_3.9x8.7mm_P1.27mm" H 1650 6750 50  0001 C CNN
 F 3 "http://www.ti.com/lit/ds/symlink/tl071.pdf" H 1750 6850 50  0001 C CNN
